File: main.brd (EAGLE design)
At the start: 146.5 x 85 mm, 46 parts, among them X1 ZX62D-B-5PA8

Commit message: Final version 1 changes
Parts:
- removed C1: 10uF, rcl:C0805
- added C7: 22µF, AVX_By_element14_Batch_1:CAPCP3216X180N
- added U1: 0ZCH0075AF2E, CustomParts:0ZCH
- 3V_SRC: value V_REG_LD1117VXXLD1117-SMD -> (none)
- C2: value 22uF -> 10µF; device rcl:C0805 -> AVX_By_element14_Batch_1:CAPCP6032X280N
- moved C15 11.5 mm to (5.50, 3.00)
- moved C14 7.07 mm to (-4.00, 3.00), turned to 90 degrees
- moved 3V_SRC 3.61 mm to (0.50, 3.00), turned to 0 degrees
- moved SV3 3.50 mm to (-18.0, 9.00)
- moved LLC_RX_HIGH 2.50 mm to (5.00, 9.00), turned to 180 degrees
- moved C2 1.41 mm to (-7.50, 3.00), turned to 90 degrees
- moved C3 1.00 mm to (-11.4, -24.5)
- moved C4 1.00 mm to (-14.0, -24.5)
- moved C5 1.00 mm to (-6.36, -24.5)
- moved C6 1.00 mm to (-8.91, -24.5)
- moved R11 0.50 mm to (-11.4, -16.5)
- moved R13 0.50 mm to (-14.0, -16.5)
- moved C16 0.50 mm to (9.00, -31.5)
- moved C17 0.50 mm to (6.50, -31.5)
- moved LLC_RX 0.50 mm to (4.00, 12.0)
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Connections:
- removed net INPUT_V: U$4.3, X1.1
- new net FUSE: U1.2, X1.1
- new net N$3: U$4.3, U1.1
- net 3V3: now also 3V_SRC.4, C7.1; no longer C2.1
- net GND: now also C7.2; no longer C1.2
- net VCC: now also C2.1; no longer C1.1
Routing:
- net 3V3: track 41.7 -> 23.3 mm
- net GND: track 12.5 -> 29.3 mm
- net VCC: track 17.1 -> 29.8 mm
- net RIGHT_Y: track 65.8 -> 57.9 mm
- net TX: track 35.4 -> 30.4 mm
- net SCL: track 32.6 -> 36.6 mm
- net SDA: track 28.6 -> 32.4 mm
- net RX: track 30.4 -> 28.1 mm, vias 0 -> 2
- net INPUT_V: track 1.80 -> 0.00 mm
- net RIGHT_A_SW: track 65.9 -> 67.6 mm
- net RIGHT_B_SW: track 58.3 -> 59.9 mm
- net RIGHT_B: track 6.62 -> 7.62 mm
- net RIGHT_A: track 5.76 -> 6.76 mm
- net LEFT_B: track 6.65 -> 7.65 mm
- net LEFT_A: track 5.73 -> 6.73 mm
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- added copper zone on layer 16, net 3V3
- added copper zone on layer 1, net FUSE
- added copper zone on layer 1, net N$3
- removed copper zone on layer 1, net INPUT_V
